File: BMS-Extension/foxBMS_BMS-Extension.brd (EAGLE design)
At the start: 156 x 120 mm, 220 parts, among them IC1001 AQV252G2S, IC1002 AQV252G2S, IC1003 AQV252G2S, IC1101 UA78L05ACPK, IC1102 ADUM1300ARW, IC1301 UA78L05ACPK, IC1302 LTC485CS8#PBF, IC1303 ADUM1401ARW, IC1701 ADR3425ARJZ, IC1901 UA78L05ACPK, IC1902 ADUM1402ARW, IC1903 ADUM1402ARW, IC2001 AQV25G2S, IC2002 AQV25G2S, IC2003 AQV25G2S, IC2004 AQV25G2S, IC2005 AQV25G2S, IC2006 AQV25G2S, IC801 KA7805ERTF, IC802 CPC1008N, IC803 TJA1052IT/1Y, T1001 IRLML0100TRPBF, T1002 IRLML0100TRPBF, T1003 IRLML0100TRPBF, T1501 BSS84P, T2001 IRLML0100TRPBF, T2002 IRLML0100TRPBF, T2003 IRLML0100TRPBF, T2004 IRLML0100TRPBF, T2005 IRLML0100TRPBF, T2006 IRLML0100TRPBF, T801 IRLML0100TRPBF, T901 BUK964R8-60E, X1201 43045-0400_MOLEX_4PIN, X1202 43045-0400_MOLEX_4PIN, X1203 43045-0400_MOLEX_4PIN, X1301 43045-0600_MOLEX_6PIN, X1701 43045-1200_MOLEX_12PIN, X1901 43045-1000_MOLEX_10PIN, X2001 43045-1200_MOLEX_12PIN, X801 43045-0400_MOLEX_4PIN

Commit message: Minor updates and corrections of notations, wording and bill of materials (V1.0.1). No changes in schematic and layout.
Parts:
- added U$2, U$3, U$4: (no value), foxBMS_BMS-Slave_12cell:FIDUCIAL_1MM
- R1101, R1102, R1103, R1901, R1902, R1905, R1906: value 500 -> 47
- moved R1907 2.13 mm to (52.3, 63.0), turned to 180 degrees
- moved R1904 2.10 mm to (41.5, 62.2), turned to 180 degrees
- moved R1908 2.10 mm to (52.3, 61.8), turned to 180 degrees
- moved R1903 2.10 mm to (41.5, 63.3), turned to 180 degrees
- moved D1902 0.64 mm to (40.0, 66.7)
- moved R1902 0.64 mm to (40.0, 69.7)
- moved D1901 0.63 mm to (41.3, 66.7)
- moved R1901 0.63 mm to (41.3, 69.7)
Connections:
- removed net N$24: D1901.C, IC1902.5, R1901.1
- removed net N$25: D1902.C, IC1902.6, R1902.1
- removed net N$26: D1903.C, IC1903.5, R1905.1
- removed net N$27: D1904.C, IC1903.6, R1906.1
- new net N$1111: D1903.C, IC1903.3, R1905.1
- new net N$254548: D1904.C, IC1903.4, R1906.1
- new net N$5555: D1901.C, IC1902.3, R1901.1
- new net N$7555: D1902.C, IC1902.4, R1902.1
- net ISO_GPIO_MCU_0_IN_0_EXT: now also R1901.2; no longer R1904.2
- net ISO_GPIO_MCU_0_IN_1_EXT: now also R1902.2; no longer IC1902.4, R1903.2
- net ISO_GPIO_MCU_0_IN_2_EXT: now also R1905.2; no longer IC1903.3, R1908.2
- net ISO_GPIO_MCU_0_IN_3_EXT: now also R1906.2; no longer IC1903.4, R1907.2
- net ISO_GPIO_MCU_0_OUT_0_EXT: now also IC1902.5, R1903.2; no longer R1901.2
- net ISO_GPIO_MCU_0_OUT_1_EXT: now also IC1902.6, R1904.2; no longer R1902.2
- net ISO_GPIO_MCU_0_OUT_2_EXT: now also IC1903.5, R1907.2; no longer R1905.2
- net ISO_GPIO_MCU_0_OUT_3_EXT: now also IC1903.6, R1908.2; no longer R1906.2
Routing:
- net ISO_GPIO_MCU_0_IN_3_EXT: track 55.3 -> 33.5 mm
- net ISO_GPIO_MCU_0_IN_2_EXT: track 49.6 -> 28.2 mm
- net N$1111: track 0.00 -> 18.5 mm, vias 0 -> 2
- net N$254548: track 0.00 -> 18.2 mm, vias 0 -> 2
- net ISO_GPIO_MCU_0_OUT_3_EXT: track 40.9 -> 59.1 mm
- net ISO_GPIO_MCU_0_OUT_2_EXT: track 35.6 -> 52.9 mm
- net N$27: track 16.1 -> 0.00 mm
- net N$26: track 15.6 -> 0.00 mm
- net ISO_GPIO_MCU_0_IN_1_EXT: track 35.9 -> 21.2 mm
- net ISO_GPIO_MCU_0_IN_0_EXT: track 49.6 -> 36.3 mm
- net N$7555: track 0.00 -> 12.9 mm
- net ISO_GPIO_MCU_0_OUT_1_EXT: track 30.8 -> 42.5 mm
- net N$5555: track 0.00 -> 11.7 mm
- net ISO_GPIO_MCU_0_OUT_0_EXT: track 25.3 -> 36.7 mm
- net N$25: track 11.3 -> 0.00 mm
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Other:
- board text added: "foxBMS BMS-Extension V1.0.1"
- board text removed: "Fraunhofer IISB L21585"
- board text removed: "foxBMS BMS-Master Extension V1.00"

Commit message: updated foxBMS-slave to version 2.02
Other:
- board text added: "Fraunhofer IISB L21686"
- board text added: "foxBMS BMS-Master Extension V1.0.1"
- board text removed: "foxBMS BMS-Extension V1.0.1"
Changed lines of the file:
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@@
 <layer number="27" name="tValues" color="7" fill="1" visible="no" active="yes"/>
 <layer number="28" name="bValues" color="7" fill="1" visible="no" active="yes"/>
-<layer number="29" name="tStop" color="7" fill="3" visible="yes" active="yes"/>
+<layer number="29" name="tStop" color="7" fill="3" visible="no" active="yes"/>
 <layer number="30" name="bStop" color="7" fill="6" visible="no" active="yes"/>
 <layer number="31" name="tCream" color="7" fill="4" visible="no" active="yes"/>
@@
 <text x="12.827" y="-18.796" size="0.7112" layer="25" font="vector" rot="R180">+3.3V</text>
 <text x="57.785" y="-18.796" size="0.7112" layer="25" font="vector" rot="R180">+3.3V</text>
+<text x="114.8715" y="-17.4625" size="0.8128" layer="1" font="vector">Fraunhofer IISB
+L21686</text>
 <text x="153.035" y="9.2075" size="0.8128" layer="1" font="vector">TOP</text>
 <text x="149.225" y="9.2075" size="0.8128" layer="16" font="vector" rot="MR0">BOT</text>
+<text x="114.8715" y="-17.4625" size="0.8128" layer="29" font="vector">Fraunhofer IISB
+L21686</text>
 <polygon width="0.2032" layer="25">
 <vertex x="87.1245" y="-13.2715"/>
@@
 <text x="89.2175" y="90.805" size="0.7112" layer="25">X2001</text>
 <text x="112.7125" y="90.805" size="0.7112" layer="25">X1701</text>
-<text x="88.5825" y="-12.7" size="0.8128" layer="25">foxBMS BMS-Extension V1.0.1</text>
+<text x="88.5825" y="-12.7" size="0.8128" layer="25">foxBMS BMS-Master Extension V1.0.1</text>
 <text x="139.7" y="-17.78" size="1.778" layer="25">foxBMS.org</text>
 <polygon width="0.0254" layer="25">
