File: BMS-Extension/foxBMS_BMS-Extension.sch (EAGLE design)
At the start: 219 parts, among them IC1001 AQV252G2S, IC1002 AQV252G2S, IC1003 AQV252G2S, IC1101 UA78L05ACPK, IC1102 ADUM1300ARW, IC1301 UA78L05ACPK, IC1302 LTC485CS8#PBF, IC1303 ADUM1401ARW, IC1701 ADR3425ARJZ, IC1901 UA78L05ACPK, IC1902 ADUM1402ARW, IC1903 ADUM1402ARW, IC2001 AQV25G2S, IC2002 AQV25G2S, IC2003 AQV25G2S, IC2004 AQV25G2S, IC2005 AQV25G2S, IC2006 AQV25G2S, IC801 KA7805ERTF, IC802 CPC1008N, IC803 TJA1052IT/1Y, T1001 IRLML0100TRPBF, T1002 IRLML0100TRPBF, T1003 IRLML0100TRPBF, T1501 BSS84P, T2001 IRLML0100TRPBF, T2002 IRLML0100TRPBF, T2003 IRLML0100TRPBF, T2004 IRLML0100TRPBF, T2005 IRLML0100TRPBF, T2006 IRLML0100TRPBF, T801 IRLML0100TRPBF, T901 BUK964R8-60E, X1201 43045-0400_MOLEX_4PIN, X1202 43045-0400_MOLEX_4PIN, X1203 43045-0400_MOLEX_4PIN, X1301 43045-0600_MOLEX_6PIN, X1701 43045-1200_MOLEX_12PIN, X1901 43045-1000_MOLEX_10PIN, X2001 43045-1200_MOLEX_12PIN, X801 43045-0400_MOLEX_4PIN

Commit message: updated foxBMS-slave to version 2.02
Other:
- note added: "Connectors to Basic Board"
- note added: "Please Note: As the foxBMS BMS-Master was designed as one unit, the schematic of BMS-Master Basic or Extension may include blank pages."
- note removed: "Connectors to BMS-Master"
- note removed: "This page was intentionally left blank."
Changed lines of the file:
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@@
 <setting verticaltext="up"/>
 </settings>
-<grid distance="0.1" unitdist="inch" unit="inch" style="lines" multiple="1" display="no" altdistance="0.01" altunitdist="inch" altunit="inch"/>
+<grid distance="100" unitdist="mil" unit="mil" style="lines" multiple="1" display="yes" altdistance="10" altunitdist="mil" altunit="mil"/>
 <layers>
 <layer number="1" name="Top" color="4" fill="1" visible="no" active="no"/>
@@
 <attributes>
 <attribute name="AUTHOR" value="Fraunhofer IISB foxBMS Team"/>
-<attribute name="REL-DATE" value="2017-05-09"/>
-<attribute name="TITLE" value="foxBMS BMS-Extension"/>
+<attribute name="REL-DATE" value="2017-04-13"/>
+<attribute name="TITLE" value="foxBMS BMS-Master Extension"/>
 <attribute name="VERSION" value="1.0.1"/>
 </attributes>
@@
 <wire x1="215.9" y1="238.76" x2="152.4" y2="238.76" width="0.1524" layer="105"/>
 <wire x1="152.4" y1="238.76" x2="152.4" y2="259.08" width="0.1524" layer="105"/>
+<text x="20.32" y="5.08" size="2.54" layer="105">Please Note:
+As the foxBMS BMS-Master was designed as one unit, the schematic of BMS-Master Basic or Extension may include blank pages.</text>
 </plain>
 <instances>
@@
 <plain>
 <text x="335.534" y="24.13" size="2.54" layer="105">SUPPLY_0</text>
-<text x="307.34" y="35.56" size="2.54" layer="105">This page was intentionally left blank. </text>
 </plain>
 <instances>
@@
 <plain>
 <text x="335.534" y="24.13" size="2.54" layer="105">SUPPLY_1</text>
-<text x="307.34" y="35.56" size="2.54" layer="105">This page was intentionally left blank. </text>
 </plain>
 <instances>
@@
 <plain>
 <text x="335.788" y="24.13" size="2.54" layer="105">MCU_0 (PRIMARY)</text>
-<text x="307.34" y="35.56" size="2.54" layer="105">This page was intentionally left blank. </text>
 </plain>
 <instances>
@@
 <plain>
 <text x="335.788" y="24.13" size="2.54" layer="105">MCU_1 (SECONDARY)</text>
-<text x="307.34" y="35.56" size="2.54" layer="105">This page was intentionally left blank. </text>
 </plain>
 <instances>
@@
 <plain>
 <text x="336.042" y="24.13" size="2.54" layer="105">MCU_0 to MCU_1 Isolated Interface (SPI)</text>
-<text x="307.34" y="35.56" size="2.54" layer="105">This page was intentionally left blank. </text>
 </plain>
 <instances>
@@
 <plain>
 <text x="335.534" y="24.13" size="2.54" layer="105">BENDER Isometer Interface</text>
-<text x="307.34" y="35.56" size="2.54" layer="105">This page was intentionally left blank. </text>
 </plain>
 <instances>
@@
 <plain>
 <text x="336.042" y="24.13" size="2.54" layer="105">Isolated USB MCU_0 + MCU_1</text>
-<text x="307.34" y="35.56" size="2.54" layer="105">This page was intentionally left blank. </text>
 </plain>
 <instances>
@@
 <plain>
 <text x="336.296" y="24.384" size="2.54" layer="105">BMS-Interface Interface</text>
-<text x="307.34" y="35.56" size="2.54" layer="105">This page was intentionally left blank. </text>
 </plain>
 <instances>
@@
 <plain>
 <text x="335.788" y="24.13" size="2.54" layer="105">8MB SDRAM</text>
-<text x="307.34" y="35.56" size="2.54" layer="105">This page was intentionally left blank. </text>
 </plain>
 <instances>
@@
 </sheet>
 <sheet>
-<description>Connector BMS-Master to BMS-Extension</description>
 <plain>
-<text x="336.042" y="24.13" size="2.54" layer="105">Connectors to BMS-Master</text>
+<text x="336.042" y="24.13" size="2.54" layer="105">Connectors to Basic Board</text>
 </plain>
 <instances>
