File: BMS-Interface/foxBMS_BMS-Interface.brd (EAGLE design)
At the start: 50 x 100 mm, 44 parts, among them IC301 LTC6820HMS#PBF, IC401 LTC6820HMS#PBF, T501 HX1188NL, T502 HX1188NL, X1 43045-0406_MOLEX_4PIN, X2 43045-0406_MOLEX_4PIN

Commit message: Minor updates and corrections of notations, wording and bill of materials (V1.0.1). No changes in schematic and layout.
Parts:
- added U$1, U$2: (no value), foxBMS_BMS-Slave_12cell:FIDUCIAL_1MM
Other:
- board text added: "foxBMS BMS-Interface V1.0.1"
- board text removed: "Fraunhofer IISB L21586"
- board text removed: "foxBMS BMS-Interface V1.00"
Changed lines of the file:
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@@
 <layers>
 <layer number="1" name="Top" color="4" fill="1" visible="yes" active="yes"/>
-<layer number="2" name="GND" color="1" fill="3" visible="yes" active="yes"/>
+<layer number="2" name="GND" color="1" fill="3" visible="no" active="yes"/>
 <layer number="3" name="Route3" color="4" fill="3" visible="yes" active="yes"/>
 <layer number="4" name="Route4" color="1" fill="4" visible="no" active="no"/>
@@
 <layer number="250" name="Descript" color="3" fill="1" visible="yes" active="yes"/>
 <layer number="251" name="SMDround" color="7" fill="1" visible="no" active="yes"/>
+<layer number="253" name="Insertarea2" color="7" fill="1" visible="yes" active="yes"/>
 <layer number="254" name="OrgLBR" color="13" fill="1" visible="no" active="yes"/>
+<layer number="255" name="HELP" color="11" fill="1" visible="yes" active="yes"/>
 </layers>
 <board>
@@
 <vertex x="41.3004" y="84.1248"/>
 </polygon>
-<text x="40.5384" y="81.2292" size="0.8128" layer="25" rot="R90">foxBMS BMS-Interface V1.00</text>
-<text x="47.3964" y="29.1084" size="0.8128" layer="1" rot="R90">Fraunhofer IISB
-L21586</text>
-<text x="47.3964" y="29.1084" size="0.8128" layer="29" rot="R90">Fraunhofer IISB
-L21586</text>
+<text x="40.5384" y="81.2292" size="0.8128" layer="25" rot="R90">foxBMS BMS-Interface V1.0.1</text>
 <text x="48.768" y="84.4296" size="1.778" layer="25" rot="R90">foxBMS.org</text>
 <text x="1.524" y="84.1248" size="1.778" layer="26" rot="SMR90">foxBMS.org</text>
@@
 <attribute name="NAME" x="37.0332" y="43.8912" size="0.7112" layer="25" font="vector" ratio="10" align="center"/>
 </element>
+<element name="U$1" library="foxBMS_BMS-Slave_12cell" package="FIDUCIAL_1MM" value="" x="2.1336" y="10.3632"/>
+<element name="U$2" library="foxBMS_BMS-Slave_12cell" package="FIDUCIAL_1MM" value="" x="35.9664" y="97.2312"/>
 </elements>
 <signals>
@@
 <vertex x="22.9024" y="74.9384"/>
 <vertex x="23.3172" y="74.5236"/>
-<vertex x="50" y="74.6524"/>
+<vertex x="50" y="74.5236"/>
 <vertex x="49.9872" y="77.1144"/>
 <vertex x="50" y="100"/>

Commit message: updated foxBMS-slave to version 2.02
Parts:
- removed C501, C503: 1uF, custom_passiv:0603
- removed T501, T502: HX1188NL, 0_LES_TRANSFORMER.SMD:TR_SMD_SOIC-16_(12,70MMX9,53MMX5,97MM)_R_PULSE_REV01
- added TR501, TR502: HM2102NL, transformer_custom:HM2102NL
- R405: value OPT: 0R -> 0R
- R406: value OPT: 0R -> N/A
- moved U$1 91.2 mm to (36.0, 95.0)
- moved U$2 76.8 mm to (5.00, 27.0)
- moved C504 12.5 mm to (35.7, 57.5)
- moved R502 12.2 mm to (35.7, 54.6)
- moved C502 8.57 mm to (14.4, 57.5)
- moved R501 8.19 mm to (14.4, 54.6)
Connections:
- removed net GND_EXT_0: C501.1
- removed net GND_EXT_1: C503.1
- removed net N$22: C503.2, T502.15
- removed net N$23: C502.2, T501.7
- removed net N$24: C501.2, T501.10
- new net N$2: C502.2, TR501.11
- net N$21: now also TR502.8; no longer T502.2
- net PRIMARY_OUT+_P: now also TR501.3; no longer T501.11
- net PRIMARY_OUT-_N: now also TR501.1; no longer T501.9
- net PRIMARY_OUT_N: now also TR501.12; no longer T501.8
- net PRIMARY_OUT_P: now also TR501.10; no longer T501.6
- net SECONDARY_OUT+_P: now also TR502.6; no longer T502.16
- net SECONDARY_OUT-_N: now also TR502.4; no longer T502.14
- net SECONDARY_OUT_N: now also TR502.9; no longer T502.3
- net SECONDARY_OUT_P: now also TR502.7; no longer T502.1
Routing:
- net SECONDARY_OUT_P: track 29.3 -> 15.1 mm
- net SECONDARY_OUT_N: track 29.1 -> 15.6 mm
- net SECONDARY_OUT-_N: track 18.7 -> 32.1 mm
- net PRIMARY_OUT_N: track 23.5 -> 15.1 mm
- net PRIMARY_OUT_P: track 23.6 -> 15.6 mm
- net SECONDARY_OUT+_P: track 17.7 -> 25.3 mm, vias 1 -> 2
- net PRIMARY_OUT+_P: track 17.3 -> 23.3 mm
- net PRIMARY_OUT-_N: track 19.5 -> 23.9 mm, vias 1 -> 2
- net BMS-INTERFACE_1_SPI_MOSI: track 44.4 -> 41.9 mm, vias 0 -> 2
- net GND_EXT_0: track 2.50 -> 0.00 mm, vias 1 -> 0
- net N$22: track 1.89 -> 0.00 mm
- net N$24: track 1.89 -> 0.00 mm
- net N$2: track 0.00 -> 1.85 mm
- net N$23: track 1.83 -> 0.00 mm
- net GND_EXT_1: track 1.12 -> 0.00 mm, vias 1 -> 0
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- removed copper zone on layer 2, net GND_EXT_0
- removed copper zone on layer 2, net GND_EXT_1
Other:
- board text added: "Fraunhofer IISB L21586"
- board text added: "foxBMS BMS-Interface V1.1.0"
- board text removed: "foxBMS BMS-Interface V1.0.1"
