File: BMS-Interface/foxBMS_BMS-Interface.sch (EAGLE design)
At the start: 44 parts, among them IC301 LTC6820HMS#PBF, IC401 LTC6820HMS#PBF, T501 HX1188NL, T502 HX1188NL, X1 43045-0406_MOLEX_4PIN, X2 43045-0406_MOLEX_4PIN

Commit message: updated foxBMS-slave to version 2.02
Parts:
- removed C501, C503: 1uF, custom_passiv:C_NP0_0603
- removed T501, T502: HX1188NL, 0_LES_TRANSFORMER.SMD:HX1188NL
- added TR501, TR502: HM2102NL, transformer_custom:HM2102NL
- R405: value OPT: 0R -> 0R
- R406: value OPT: 0R -> N/A
Connections:
- removed net GND_EXT_0: C501.1
- removed net GND_EXT_1: C503.1
- removed net N$22: C503.2, T502-TRANSMIT.CMT
- removed net N$23: C502.2, T501-RECEIVE.CT
- removed net N$24: C501.2, T501-RECEIVE.CMT
- new net N$2: C502.2, TR501-1.CMT
- net N$21: now also TR502-2.CMT; no longer T502-TRANSMIT.CT
- net PRIMARY_OUT+_P: now also TR501-1.D-; no longer T501-RECEIVE.X+
- net PRIMARY_OUT-_N: now also TR501-1.D+; no longer T501-RECEIVE.X-
- net PRIMARY_OUT_N: now also TR501-1.X+; no longer T501-RECEIVE.D-
- net PRIMARY_OUT_P: now also TR501-1.X-; no longer T501-RECEIVE.D+
- net SECONDARY_OUT+_P: now also TR502-2.D-; no longer T502-TRANSMIT.X+
- net SECONDARY_OUT-_N: now also TR502-2.D+; no longer T502-TRANSMIT.X-
- net SECONDARY_OUT_N: now also TR502-2.X+; no longer T502-TRANSMIT.D-
- net SECONDARY_OUT_P: now also TR502-2.X-; no longer T502-TRANSMIT.D+
