File: BMS-Master/foxBMS_BMS-Master.sch (EAGLE design)
At the start: 314 parts, among them IC1001 AQV252G2S, IC1002 AQV252G2S, IC1003 AQV252G2S, IC1004 AQV252G2S, IC1005 AQV252G2S, IC1006 AQV252G2S, IC1101 UA78L05ACPK, IC1102 ADUM1300ARW, IC1103 ADUM1300ARW, IC1401 IP4220CZ6, IC1402 FT231XS-R, IC1403 ADUM1401ARW, IC1404 IP4220CZ6, IC1405 FT231XS-R, IC1406 ADUM1401ARW, IC1501 AT25128B-SSHL-T, IC1801 IS42S16400J-5TL, IC201 LM1085IS-5.0/NOPB, IC202 MURATA_NCS6S1205C, IC301 LM1085IS-5.0/NOPB, IC302 RS-2405D/H2, IC401 ADR3425ARJZ, IC402 STM32F429IIT6, IC501 STM32F429VIT6, IC601 ADUM1401ARW, IC701 UA78L05ACPK, IC702 ADUM1301ARW, IC801 KA7805ERTF, IC802 TJA1052IT/1Y, IC803 CPC1008N, IC901 LM317MBSTT3G, IC902 CPC1008N, IC903 CPC1008N, IC904 CPC1008N, IC905 CPC1008N, Q401 7B-8.000MAAJ-T, Q501 7B-8.000MAAJ-T, T1001 IRLML0100TRPBF, T1002 IRLML0100TRPBF, T1003 IRLML0100TRPBF, T1004 IRLML0100TRPBF, T1005 IRLML0100TRPBF, T1006 IRLML0100TRPBF, T201 TISP40XXH1BJ, T401 BSS84P, T501 BSS84P, T701 IRLML0100TRPBF, T801 IRLML0100TRPBF, T901 BUK964R8-60E, T902 IRLML0100TRPBF, T903 IRLML0100TRPBF, X1201 43045-0400_MOLEX_4PIN, X1202 43045-0400_MOLEX_4PIN, X1203 43045-0400_MOLEX_4PIN, X1204 43045-0400_MOLEX_4PIN, X1205 43045-0400_MOLEX_4PIN, X1206 43045-0400_MOLEX_4PIN, X1401 MINI-USB-2.0, X1402 MINI-USB-2.0, X1601 43045-1600_MOLEX_16PIN, X201 43045-0600_MOLEX_6PIN, X402 MA02-1, X403 SAMTEC_FTS_20POL_HEADER_VERTI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, X501 MA02-1, X502 SAMTEC_FTS_20POL_HEADER_VERTI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, X701 43045-0400_MOLEX_4PIN, X801 43045-0400_MOLEX_4PIN, X901 43045-0200_MOLEX_2PIN, X902 MA02-1SMALL_PINS_OUTLINE

Commit message: updated foxBMS-slave to version 2.02
Other:
- note added: "Connectors to Extension Board"
- note added: "Please Note: As the BMS-Master was designed as one unit, the schematic of BMS-Master Basic or Extension may include blank pages."
- note removed: "Connectors to BMS-Extension"
- note removed: "This page was intentionally left blank."
Changed lines of the file:
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@@
 <attributes>
 <attribute name="AUTHOR" value="Fraunhofer IISB foxBMS Team"/>
-<attribute name="REL-DATE" value="2017-05-09"/>
-<attribute name="TITLE" value="foxBMS BMS-Master"/>
+<attribute name="REL-DATE" value="2017-04-13"/>
+<attribute name="TITLE" value="foxBMS BMS-Master Basic"/>
 <attribute name="VERSION" value="1.0.1"/>
 </attributes>
@@
 <wire x1="215.9" y1="238.76" x2="152.4" y2="238.76" width="0.1524" layer="105"/>
 <wire x1="152.4" y1="238.76" x2="152.4" y2="259.08" width="0.1524" layer="105"/>
+<text x="30.48" y="5.08" size="2.54" layer="105">Please Note:
+As the BMS-Master was designed as one unit, the schematic of BMS-Master Basic or Extension may include blank pages.</text>
 </plain>
 <instances>
@@
 <plain>
 <text x="335.788" y="24.13" size="2.54" layer="105">Isolated RS485</text>
-<text x="307.34" y="35.56" size="2.54" layer="105">This page was intentionally left blank. </text>
 </plain>
 <instances>
@@
 <plain>
 <text x="336.042" y="24.384" size="2.54" layer="105">Analog Inputs</text>
-<text x="307.34" y="35.56" size="2.54" layer="105">This page was intentionally left blank. </text>
 </plain>
 <instances>
@@
 <plain>
 <text x="336.296" y="24.13" size="2.54" layer="105">Isolated GPIO 4x In /  4x Out</text>
-<text x="307.34" y="35.56" size="2.54" layer="105">This page was intentionally left blank. </text>
 </plain>
 <instances>
@@
 <plain>
 <text x="336.296" y="24.13" size="2.54" layer="105">Isolated Normally Open Contacts</text>
-<text x="307.34" y="35.56" size="2.54" layer="105">This page was intentionally left blank. </text>
 </plain>
 <instances>
@@
 </sheet>
 <sheet>
-<description>Connector BMS-Master to BMS-Extension</description>
+<description>Basic to Extension Connector</description>
 <plain>
-<text x="336.296" y="24.13" size="2.54" layer="105">Connectors to BMS-Extension</text>
+<text x="336.296" y="24.13" size="2.54" layer="105">Connectors to Extension Board</text>
 </plain>
 <instances>
