File: BMS-Slave/foxBMS_BMS-Slave_12cell.sch (EAGLE design)
At the start: 369 parts, among them IC1001 ADG728BRUZ, IC1002 ADG728BRUZ, IC1003 LTC6255CS6, IC1004 LTC6255CS6, IC1005 ADG728BRUZ, IC1101 PCA8574TS, IC1201 PCA8574TS, IC1301 24AA02UID, IC1302 MCP9800A0T-M/OT, IC1401 24AA02UID, IC1402 MCP9800A0T-M/OT, IC201 0_LES_BATTERIE-MANAGEMENT.SMD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, IC301 0_LES_BATTERIE-MANAGEMENT.SMD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, IC801 ACPL-247-500E, IC802 ACPL-247-500E, IC803 ACPL-247-500E, IC901 ADG728BRUZ, IC902 ADG728BRUZ, IC903 LTC6255CS6, IC904 LTC6255CS6, IC905 ADG728BRUZ, T201 PBHV8115Z, T301 PBHV8115Z, T701 NX2301P, T702 NX2301P, T703 NX2301P, T704 NX2301P, T705 NX2301P, T706 NX2301P, T707 NX2301P, T708 NX2301P, T709 NX2301P, T710 NX2301P, T711 NX2301P, T712 NX2301P, X1501 MA09-2, X1502 MA09-2, X1503 43045-2400_MOLEX_24PIN, X1504 MA05-2, X1505 MA05-2, X1506 43045-1600_MOLEX_16PIN, X1507 43045-1600_MOLEX_16PIN, X1508 MA10-2, X1509 43045-0200_MOLEX_2PIN, X1510 43045-0200_MOLEX_2PIN, X1511 43045-0200_MOLEX_2PIN, X1512 43045-0200_MOLEX_2PIN

Commit message: updated foxBMS-slave to version 2.1.0
Parts:
- removed TP202, TP208, TP302, TP308: CUSTOM_PAD_PAD_2.0X1.5MM, foxBMS_BMS-Slave_12cell:CUSTOM_PAD_PAD_2.0X1.5MM
- added C1601: 1,00µF_0805_25V_X7R_KEMET, 0_LES_KAPAZITAET.SMD.MLCC:1,00µF_0805_25V_X7R_KEMET
- added C1602, C1603: 10µF_1210_25V_X7R, 0_LES_KAPAZITAET.SMD.MLCC.KEMET:10µF_1210_25V_X7R
- added C1604: 100nF, 20%, 16V, foxBMS_BMS-Slave_12cell:100NF_0603_16V_X7R_KEMET
- added C1605: 1uF, 20%, 16V, foxBMS_BMS-Slave_12cell:1,00µF_0603_16V_X7R_KEMET
- added C1606: 470PF_0805_50V_X7R_KEMET, 0_LES_KAPAZITAET.SMD.MLCC:470PF_0805_50V_X7R_KEMET
- added C1607: 4,7NF_1812, 0_LES_KAPAZITAET.SMD.MLCC.KEMET_custom:4,7NF_1812
- added C1608, C1609, C1610: 4,70µF_1206_25V_X7R_KEMET, 0_LES_KAPAZITAET.SMD.MLCC:4,70µF_1206_25V_X7R_KEMET
- added D1601, D1603: DI_DFLS1100, diodes_custom:DI_DFLS1100
- added D1602: DI_DFLZ36, diodes_custom:DI_DFLZ36
- added D1604: DI_PDS3200, diodes_custom:DI_PDS3200
- added D1605: MMSZ5263B, L21596_V1.0:MMSZ524CBT1
- added D202, D302: SMAJ60CA_VISHAY, foxBMS_BMS-Slave_12cell:SMAJ60CA_VISHAY
- added F1601: 1,250A_LITTELFUSE_466_1206, foxBMS_BMS-Slave_12cell:1,250A_LITTELFUSE_466_1206
- added IC1601: LT8302, linear_custom:LT8302
- added L1601: WE-74404042100, inductor_custom:WE-74404042100
- added R1302, R1402: 10,0K_0603_R_VISHAY_1%_TK100_REV_01, foxBMS_BMS-Slave_12cell:10,0K_0603_R_VISHAY_1%_TK100_REV_01
- added R1601: 390K_0603_R_VISHAY_1%_TK100_REV_01, 0_LES_WIDERSTAND.SMD.CHIP.DICKSCHICHT:390K_0603_R_VISHAY_1%_TK100_REV_01
- added R1602: 86,6K_0603_R_VISHAY_1%_TK100_REV_01, 0_LES_WIDERSTAND.SMD.CHIP.DICKSCHICHT:86,6K_0603_R_VISHAY_1%_TK100_REV_01
- added R1603: 39,0R_0805_R_VISHAY_1%_TK100_REV_01, 0_LES_WIDERSTAND.SMD.CHIP.DICKSCHICHT:39,0R_0805_R_VISHAY_1%_TK100_REV_01
- added R1604: DUMMY_R_CHIP_0603_R_VISHAY, 0_LES_WIDERSTAND.SMD.CHIP.DICKSCHICHT:DUMMY_R_CHIP_0603_R_VISHAY
- added R1605: 127K_0603_R_VISHAY_1%_TK100_REV_01, 0_LES_WIDERSTAND.SMD.CHIP.DICKSCHICHT:127K_0603_R_VISHAY_1%_TK100_REV_01
- added R1606: 10,0K_0603_R_VISHAY_1%_TK100_REV_01, 0_LES_WIDERSTAND.SMD.CHIP.DICKSCHICHT:10,0K_0603_R_VISHAY_1%_TK100_REV_01
- added R223, R323: 1.2k, 10%, 1/10W, foxBMS_BMS-Slave_12cell:1,20K_0603_R_VISHAY_1%_TK100_REV_01
- added TP1601, TP1602, TP1603: CUSTOM_PAD_PAD_2.0X1.5MM, foxBMS_BMS-Slave_12cell:CUSTOM_PAD_PAD_2.0X1.5MM
- added TR1601: WE_750313457, transformer_custom:WE_750313457
- added X1513, X1514: 43045-0200_MOLEX_2PIN, foxBMS_BMS-Slave_12cell:43045-0200_MOLEX_2PIN
- added X1515: MA02-2_TH, custom_connector:MA02-2_TH
- added X1601: MA02-1_TH, custom_connector:MA02-1_TH
- D201, D301: value SMAJ60CA_VISHAY -> DI_DFLS1100; device foxBMS_BMS-Slave_12cell:SMAJ60CA_VISHAY -> diodes_custom:DI_DFLS1100
- IC1301, IC1401: value 24AA02UID -> M24M02-DR; device foxBMS_BMS-Slave_12cell:24AA02UID -> eeprom_custom:M24M02-DR
- R201, R301: value 100R, 1%, 1/10W -> 0,00R_0805_R_VISHAY_REV_01; device foxBMS_BMS-Slave_12cell:100R_0805_R_VISHAY_1%_TK100_REV_01 -> 0_LES_WIDERSTAND.SMD.CHIP.DICKSCHICHT:0,00R_0805_R_VISHAY_REV_01
- R203, R303: value 120R, 1%, 1/10W -> 100R, 1%, 1/10W; device foxBMS_BMS-Slave_12cell:120R_0603_R_VISHAY_1%_TK100_REV_01 -> foxBMS_BMS-Slave_12cell:100R_0805_R_VISHAY_1%_TK100_REV_01
- R204, R304: value 270R, 1%, 1/10W -> 120R, 1%, 1/10W; device foxBMS_BMS-Slave_12cell:270R_0603_R_VISHAY_1%_TK100_REV_01 -> foxBMS_BMS-Slave_12cell:120R_0603_R_VISHAY_1%_TK100_REV_01
- R205, R305: value 820R, 1%, 1/10W -> 330R, 1%, 1/10W; device foxBMS_BMS-Slave_12cell:820R_0603_R_VISHAY_1%_TK100_REV_01 -> 0_LES_WIDERSTAND.SMD.CHIP.DICKSCHICHT:330R_0603_R_VISHAY_1%_TK100_REV_01
- R206, R306: value 120R, 1%, 1/10W -> 820R, 1%, 1/10W; device foxBMS_BMS-Slave_12cell:120R_0603_R_VISHAY_1%_TK100_REV_01 -> foxBMS_BMS-Slave_12cell:820R_0603_R_VISHAY_1%_TK100_REV_01
- R207, R307: value 1.21k, 1%, 1/10W -> 120R, 1%, 1/10W; device foxBMS_BMS-Slave_12cell:1,21K_0603_R_VISHAY_1%_TK100_REV_01 -> foxBMS_BMS-Slave_12cell:120R_0603_R_VISHAY_1%_TK100_REV_01
- R208, R308: value OPT -> 1.21k, 1%, 1/10W; device foxBMS_BMS-Slave_12cell:0,00R_0603_R_VISHAY_REV_01 -> foxBMS_BMS-Slave_12cell:1,21K_0603_R_VISHAY_1%_TK100_REV_01
- R209, R211, R213, R215, R217, R309, R311, R313, R315, R317: value 0R -> OPT
- R210, R212, R214, R216, R220, R310, R312, R314, R316, R320: value OPT -> 0R
- R218, R318: value 1M, 10%, 1/10W -> 0R; device foxBMS_BMS-Slave_12cell:1,00M_0603_R_VISHAY_1%_TK100_REV_01 -> foxBMS_BMS-Slave_12cell:0,00R_0603_R_VISHAY_REV_01
- R219, R319: value 0R -> 1M, 10%, 1/10W; device foxBMS_BMS-Slave_12cell:0,00R_0603_R_VISHAY_REV_01 -> foxBMS_BMS-Slave_12cell:1,00M_0603_R_VISHAY_1%_TK100_REV_01
- R221, R321: value 1.2k, 10%, 1/10W -> OPT; device foxBMS_BMS-Slave_12cell:1,20K_0603_R_VISHAY_1%_TK100_REV_01 -> foxBMS_BMS-Slave_12cell:0,00R_0603_R_VISHAY_REV_01
- R701, R702, R703, R704, R705, R706, R707, R708, R709, R710, R711, R712, R719, R720, R721, R722, R723, R724, R725, R726, R727, R728, R729, R730: value 18R, 1%, 0.4W -> 72R, 1%; device foxBMS_BMS-Slave_12cell:18,0R_2010_R_YAGEO_5%_TK100_REV_01 -> 0_LES_WIDERSTAND.SMD.CHIP.DICKSCHICHT:68,0R_2010_R_YAGEO_5%_TK100_REV_01
- TR201, TR301: value HX1188NL -> HM2102NL; device foxBMS_BMS-Slave_12cell:HX1188NL -> transformer_custom:HM2102NL
Connections:
- removed net N$11: R705.1, R711.2
- removed net N$13: R704.1, R710.2
- removed net N$19: R703.1, R709.2
- removed net N$21: R701.1, R707.2
- removed net N$23: R702.1, R708.2
- removed net N$27: R719.1, R725.2
- removed net N$29: R720.1, R726.2
- removed net N$4: R706.1, R712.2
- removed net N$41: R721.1, R727.2
- removed net N$43: R722.1, R728.2
- removed net N$46: R723.1, R729.2
- removed net N$48: R724.1, R730.2
- new net EXT_DC_IN+: F1601.P$1, X1513.1, X1514.1, X1515.1, X1515.3
- new net EXT_DC_IN-: C1601.P$1, C1602.P$1, C1603.P$1, C1604.P$1, C1605.P$1, C1607.P$1, IC1601.GND, R1602.1, R1606.1, TP1601.MP, X1513.2, X1514.2, X1515.2, X1515.4
- new net EXT_DC_ISO+: C1608.P$2, C1609.P$2, C1610.P$2, D1604.C, D1605.K, D201.C, D202.K2, D301.C, D302.K2, R202.2, R203.1, R302.2, R303.1, X1601.1
- new net N$1254: C1602.P$2, C1603.P$2, C1606.P$2, D1602.A, IC1601.V_IN, L1601.2, R1601.2, TR1601.PIN4
- new net N$68: C1604.P$2, IC1601.EN/UVLO, R1601.1, R1602.2
- new net N$71: C1605.P$2, IC1601.INTVCC
- new net N$74: TR1601.PIN6, TR1601.PIN7
- new net N$76: D201.A, R201.2
- new net N$77: IC1601.R_REF, R1604.2, R1606.2
- new net N$79: IC1601.R_FB, R1605.1
- new net N$80: D1603.A, IC1601.SW, R1603.1, R1605.2, TR1601.PIN2
- new net N$82: IC1601.TC, R1604.1
- new net N$84: D1604.A, TR1601.PIN5
- new net N$87: C1606.P$1, R1603.2
- new net N$89: D1601.A, F1601.P$2
- new net N$91: C1601.P$2, D1601.C, L1601.1, TP1602.MP
- new net N$92: D1602.C, D1603.C
- new net N$94: IC1301.!WC, R1302.1
- new net N$95: IC1401.!WC, R1402.1
- new net N$96: D301.A, R301.2
- net +5.0V_VREG_0: now also IC1301.VCC, R1302.2, R219.2, R223.2; no longer IC1301PWR.VCC, R218.2, R220.2
- net +5.0V_VREG_1: now also IC1401.VCC, R1402.2, R319.2, R323.2; no longer IC1401PWR.VCC, R318.2, R320.2
- net CELL0_FEEDBACK+: now also R712.2
- net CELL10_FEEDBACK+: now also R726.2
- net CELL11_FEEDBACK+: now also R725.2
- net CELL1_FEEDBACK+: now also R711.2
- net CELL2_FEEDBACK+: now also R710.2
- net CELL3_FEEDBACK+: now also R709.2
- net CELL4_FEEDBACK+: now also R708.2
- net CELL5_FEEDBACK+: now also R707.2
- net CELL6_FEEDBACK+: now also R730.2
- net CELL7_FEEDBACK+: now also R729.2
- net CELL8_FEEDBACK+: now also R728.2
- net CELL9_FEEDBACK+: now also R727.2
- net FUSED_CELL_0+: now also R705.1
- net FUSED_CELL_0-: now also R706.1
- net FUSED_CELL_1+: now also R704.1
- net FUSED_CELL_10+: now also R719.1
- net FUSED_CELL_2+: now also R703.1
- net FUSED_CELL_3+: now also R702.1
- net FUSED_CELL_4+: now also R701.1
- net FUSED_CELL_5+: now also R724.1
- net FUSED_CELL_6+: now also R723.1
- net FUSED_CELL_7+: now also R722.1
- net FUSED_CELL_8+: now also R721.1
- net FUSED_CELL_9+: now also R720.1
- net FUSED_VBAT+: no longer D201.K2, D301.K2, R202.2, R302.2
- net FUSED_VBAT-: now also C1607.P$2, C1608.P$1, C1609.P$1, C1610.P$1, D1605.A, D202.K1, D302.K1, IC1301.E2, IC1301.VSS, IC1401.E2, IC1401.VSS, R205.1, R208.1, R220.1, R305.1, R308.1, R320.1, TP1603.MP, TR1601.PIN8, X1601.2; no longer D201.K1, D301.K1, IC1301PWR.VSS, IC1401PWR.VSS, R204.1, R207.1, R219.1, R304.1, R307.1, R319.1
- net GLOBAL-BALANCING-FEEDBACK: now also R214.1, R314.1; no longer R213.1, R313.1
- net N$12: now also R206.2; no longer R205.2
- net N$14: now also TR301-1.CMT; no longer TR301-TRANSMIT.CMT
- net N$15: now also TR301-2.CMT; no longer TR301-RECEIVE.CMT
- net N$17: now also C202.P$1, R203.2; no longer C201.P$1, R201.2
- net N$24: now also C302.P$1, R303.2; no longer C301.P$1, R301.2
- net N$25: now also C301.P$1; no longer C302.P$1
- net N$33: now also R306.2; no longer R305.2
- net N$34: now also R205.2; no longer R204.2
- net N$38: now also R305.2; no longer R304.2
- net N$40: now also R316.2; no longer R314.2
- net N$5: now also TR201-1.CMT; no longer TR201-TRANSMIT.CMT
- net N$7: now also C201.P$1; no longer C202.P$1
- net N$9: now also TR201-2.CMT; no longer TR201-RECEIVE.CMT
- net PRIMARY-GPIO0: now also R210.2; no longer R208.2
- net PRIMARY-GPIO1: now also R212.2; no longer R210.2
- net PRIMARY-GPIO1-OPT: now also R209.1; no longer R208.1
- net PRIMARY-GPIO2-OPT: now also R211.1; no longer R210.1
- net PRIMARY-GPIO3: now also R216.2; no longer R214.2
- net PRIMARY-GPIO3-OPT: now also R213.1; no longer R212.1
- net PRIMARY-GPIO4: now also R218.2; no longer R216.2
- net PRIMARY-GPIO4-OPT: now also R215.1; no longer R214.1
- net PRIMARY-GPIO5: now also R214.2; no longer R212.2
- net PRIMARY-GPIO5-OPT: now also R217.1; no longer R216.1
- net PRIMARY-ICMP: now also R206.1, R208.2; no longer R205.1, R207.2
- net PRIMARY-ICMP1: now also R306.1, R308.2; no longer R305.1, R307.2
- net PRIMARY-IN+: now also TR201-2.D+; no longer TR201-RECEIVE.D+
- net PRIMARY-IN-: now also TR201-2.D-; no longer TP202.MP, TR201-RECEIVE.D-
- net PRIMARY-IN_N1: now also R204.2, TR201-2.X-; no longer R203.2, TR201-RECEIVE.X-
- net PRIMARY-IN_P1: now also R204.1, TR201-2.X+; no longer R203.1, TR201-RECEIVE.X+
- net PRIMARY-MUX-DATA_TEMP: now also R210.1; no longer R209.1
- net PRIMARY-MUX-DATA_USER: now also R212.1; no longer R211.1
- net PRIMARY-OUT+: now also TR201-1.D+; no longer TR201-TRANSMIT.D+
- net PRIMARY-OUT-: now also TR201-1.D-; no longer TP208.MP, TR201-TRANSMIT.D-
- net PRIMARY-OUT_N1: now also R207.2, TR201-1.X-; no longer R206.2, TR201-TRANSMIT.X-
- net PRIMARY-OUT_P1: now also R207.1, TR201-1.X+; no longer R206.1, TR201-TRANSMIT.X+
- net PRIMARY-SCL_0: now also IC1301.SCL, R218.1, R223.1; no longer IC1301G$1.SCL, R217.1, R222.1
- net PRIMARY-SDA_0: now also IC1301.SDA, R216.1, R222.1; no longer IC1301G$1.SDA, R215.1, R221.1
- net PRIMARY-SWTEN: now also R220.2, R221.1; no longer R219.2, R220.1
- net PRIMARY-SWTEN1: now also R320.2, R321.1; no longer R319.2, R320.1
- net PRIMARY-WDT: now also R219.1; no longer R218.1
- net SECONDARY-GPIO0: now also R310.2; no longer R308.2
- net SECONDARY-GPIO1: now also R312.2; no longer R310.2
- net SECONDARY-GPIO1-OPT: now also R309.1; no longer R308.1
- net SECONDARY-GPIO2-OPT: now also R311.1; no longer R310.1
- net SECONDARY-GPIO3-OPT: now also R313.1; no longer R312.1
- net SECONDARY-GPIO4: now also R318.2; no longer R316.2
- net SECONDARY-GPIO4-OPT: now also R315.1; no longer R314.1
- net SECONDARY-GPIO5: now also R314.2; no longer R312.2
- net SECONDARY-GPIO5-OPT: now also R317.1; no longer R316.1
- net SECONDARY-IN+: now also TR301-2.D+; no longer TR301-RECEIVE.D+
- net SECONDARY-IN-: now also TR301-2.D-; no longer TP302.MP, TR301-RECEIVE.D-
- net SECONDARY-IN_N1: now also R304.2, TR301-2.X-; no longer R303.2, TR301-RECEIVE.X-
- net SECONDARY-IN_P1: now also R304.1, TR301-2.X+; no longer R303.1, TR301-RECEIVE.X+
- net SECONDARY-MUX-DATA_TEMP: now also R310.1; no longer R309.1
- net SECONDARY-MUX-DATA_USER: now also R312.1; no longer R311.1
- net SECONDARY-OUT+: now also TR301-1.D+; no longer TR301-TRANSMIT.D+
- net SECONDARY-OUT-: now also TR301-1.D-; no longer TP308.MP, TR301-TRANSMIT.D-
- net SECONDARY-OUT_N1: now also R307.2, TR301-1.X-; no longer R306.2, TR301-TRANSMIT.X-
- net SECONDARY-OUT_P1: now also R307.1, TR301-1.X+; no longer R306.1, TR301-TRANSMIT.X+
- net SECONDARY-SCL_1: now also IC1401.SCL, R318.1, R323.1; no longer IC1401G$1.SCL, R317.1, R322.1
- net SECONDARY-SDA_1: now also IC1401.SDA, R316.1, R322.1; no longer IC1401G$1.SDA, R315.1, R321.1
- net SECONDARY-WDT: now also R319.1; no longer R318.1
Other:
- note added: "!WC: floating: write operation enabled pulled high: write operations disabled When Write Control (WC) is driven high, device select and address bytes are acknowledged, data bytes are not acknowledged."
- note added: "0x50 (see manual for MSB addressing)"
- note added: "1 MHz (max.)"
- note added: "147mA @ 5.0V 123mA @ 4.2V 118mA @ 4.0V 112mA @ 3.8V 106mA @ 3.6V"
- note added: "2.0.0"
- note added: "2.0.1"
- note added: "2.0.2"
- note added: "2.0.3"
- note added: "2.1.0"
- note added: "2017-09-04"
- note added: "400 kHz (max.)"
- note added: "Added 8-24 V isolated external power supply"
- note added: "Cell balancing control (not used on secondary)"
- note added: "EEPROM 7-bit base address 0x50 primary I²C 10100 (A17) (A16) A17, A16: MSB address bits"
- note added: "EEPROM 7-bit base address 0x50 secondary I²C 10100 (A17) (A16) A17, A16: MSB address bits"
- note added: "External Power Supply"
- note added: "Fixed isoSPI transformer CMC issue"
- note added: "Flyback Transformer"
- note added: "Fuse + Reverse Polarity Protection"
- note added: "I2C clock"
- note added: "LED on: LTC in STANDBY, REFUP or MEASURE LED off: LTC in SLEEP mode"
- note added: "LED on: LTC in STANDBY, REFUP or MEASURE mode LED off: LTC in SLEEP mode"
- note added: "LTC6804-1 LTC6811-1 Primary including power supply"
- note added: "LTC6804-1 LTC6811-1 Secondary including power supply"
- note added: "Primary LTC6804/LTC6811"
- note added: "R209: GPIO1 connected to pin header R210: GPIO1 connected to temperature MUX"
- note added: "R211: GPIO2 connected to pin header R212: GPIO2 connected to user MUX"
- note added: "R213: GPIO3 connected to pin header R214: GPIO3 connected to balancing feedback"
- note added: "R215: GPIO4 connected to pin header R216: GPIO4 connected to I2C SDA"
- note added: "R217: GPIO5 connected to pin header R218: GPIO5 connected to I2C SCL"
- note added: "R309: GPIO1 connected to pin header R310: GPIO1 connected to temperature MUX"
- note added: "R311: GPIO2 connected to pin header R312: GPIO2 connected to user MUX"
- note added: "R313: GPIO3 connected to pin header R314: GPIO3 connected to balancing feedback"
- note added: "R315: GPIO4 connected to pin header R316: GPIO4 connected to I2C SDA"
- note added: "R317: GPIO5 connected to pin header R318: GPIO5 connected to I2C SCL"
- note added: "Replaced I2C EEPROM 24AA02UID with M24M02-DR (ECC)"
- note added: "Secondary LTC6804/LTC6811"
- note added: "Snubber"
- note added: "Switched connection of balancing resistors from serial to parallel"
- note added: "Temperature Compensation"
- note added: "V_IN = 8 .. 24 V"
- note added: "battery cell supply 11 - 60 V via fuses"
- note added: "next LTC6804/LTC6811 in daisy-chain"
- note added: "optional ext. DC supply 8 - 24 V"
- note added: "previous LTC6804/LTC6811 in daisy-chain"
- note removed: "0x50"
- note removed: "139mA @ 5.0V 117mA @ 4.2V 111mA @ 4.0V 106mA @ 3.8V 100mA @ 3.6V"
- note removed: "2.00"
- note removed: "2.01"
- note removed: "2.02"
- note removed: "2.03"
- note removed: "400 kHz"
- note removed: "Cell balancing control (not used on secondary LTC6804)"
- note removed: "EEPROM 7-bit address 0x50 primary I²C 1010000"
- note removed: "EEPROM 7-bit address 0x50 secondary I²C 1010000"
- note removed: "LED on: LTC6804 in STANDBY, REFUP or MEASURE LED off: LTC6804 in SLEEP mode"
- note removed: "LED on: LTC6804 in STANDBY, REFUP or MEASURE mode LED off: LTC6804 in SLEEP mode"
- note removed: "LTC6804/11 Primary including power supply"
- note removed: "LTC6804/11 Secondary including power supply"
- note removed: "Primary LTC6804/11"
- note removed: "R210: GPIO1 connected to pin header R211: GPIO1 connected to temperature MUX"
- note removed: "R212: GPIO2 connected to pin header R213: GPIO2 connected to user MUX"
- note removed: "R214: GPIO3 connected to pin header R215: GPIO3 connected to balancing feedback"
- note removed: "R216: GPIO4 connected to pin header R217: GPIO4 connected to I2C SDA"
- note removed: "R218: GPIO5 connected to pin header R219: GPIO5 connected to I2C SCL"
- note removed: "R310: GPIO1 connected to pin header R311: GPIO1 connected to temperature MUX"
- note removed: "R312: GPIO2 connected to pin header R313: GPIO2 connected to user MUX"
- note removed: "R314: GPIO3 connected to pin header R315: GPIO3 connected to balancing feedback"
- note removed: "R316: GPIO4 connected to pin header R317: GPIO4 connected to I2C SDA"
- note removed: "R318: GPIO5 connected to pin header R319: GPIO5 connected to I2C SCL"
- note removed: "Secondary LTC6804/11"
- note removed: "Status: A"
- note removed: "battery cell supply 11 - 60V via fuses"
- note removed: "fixed isoSPI transformer CMC issue"
- note removed: "max. I2C clock"
- note removed: "next LTC6804 in daisy-chain"
- note removed: "previous LTC6804 in daisy-chain"
